File: PCB Rev B/RocketServo.kicad_pcb (KiCad board)
At the start: 2 copper layers, 60.3 x 14.6 mm, 25 parts, among them IC1 PIC12F1822-I/P, P1 Conn_01x02, P2 Conn_01x03, P3 Conn_01x02, SW1 Conn_01x02, SW2 Conn_01x02, U1 L7805, U2 TLP227GN

Commit message: Added LED1 and BattV
Parts:
- added C7: .1uF, Capacitor_SMD:C_0805_2012Metric_Pad1.18x1.45mm_HandSolder, B.Cu at (132.7, 92.1)
- added LED1: Conn_01x02, Connector_PinHeader_2.54mm:PinHeader_1x02_P2.54mm_Vertical, F.Cu at (122.6, 93.3)
- added R10: 20K, Resistor_SMD:R_0805_2012Metric_Pad1.20x1.40mm_HandSolder, B.Cu at (132.7, 88.3)
- added R11: 1K, Resistor_SMD:R_0805_2012Metric_Pad1.20x1.40mm_HandSolder, B.Cu at (132.7, 90.2)
- added R9: 270, Resistor_SMD:R_0805_2012Metric_Pad1.20x1.40mm_HandSolder, B.Cu at (132.7, 86.4)
Connections:
- IC1 pad 7: unconnected-(IC1-Pad7) -> /BattV
Routing:
- net Net-(C2-Pad1): track 20.8 -> 53.3 mm, vias 0 -> 1
- net GND: track 111.0 -> 131.4 mm, vias 18 -> 20
- net Net-(LED1-Pad2): track 0.00 -> 12.9 mm, vias 0 -> 1
- net Net-(R2-Pad2): track 38.5 -> 47.3 mm
- net Net-(IC1-Pad5): track 24.7 -> 33.4 mm
- net /BattV: track 0.00 -> 6.62 mm
- net Net-(P2-Pad1): track 41.0 -> 34.5 mm, vias 2 -> 1
- net Net-(IC1-Pad3): track 17.2 -> 20.5 mm
- net +5V: track 69.1 -> 70.4 mm, vias 2 -> 1
- removed copper zone on F.Cu, net GND
Other:
- board text added: "Rocket Servo Rev. B DMFE 2022"
- board text removed: "Rocket Servo Rev. A DMFE 2022"
