File: PCB Rev C/RocketServo.kicad_pcb (KiCad board)
At the start: 2 copper layers, 60.3 x 14.6 mm, 33 parts, among them IC1 PIC12F1822-I/SN, P1 Conn_01x02, P2 Conn_01x03, P3 Conn_01x02, SW1 SW_Push, SW2 SW_Push, U1 L7806, U2 L78L05_SOT89, U3 CPC1017N, U4 CPC1017N

Commit message: Rev C1
Parts:
- IC1: footprint Package_SO:SOIC-8_5.23x5.23mm_P1.27mm -> Package_SO:SOIC-8_3.9x4.9mm_P1.27mm
Routing:
- net /BattV: track 28.3 -> 23.6 mm
- net Net-(IC1-CLKR/C1IN1-/T1OSO/CLKOUT/OSC2/CPS3/AN3/RA4): track 25.8 -> 27.7 mm
- net /Enable*: track 31.3 -> 30.2 mm
- net Net-(IC1-Vpp/~{MCLR}/RA3): track 19.6 -> 20.8 mm
- net Net-(IC1-SRNQ/T1CKI/T1OSI/OSC1/CLKIN/RA5): track 22.0 -> 23.1 mm
- net Net-(IC1-CPS2/C1OUT/SRQ/T0CKI/FLT0/SDA/SDI/INT/MDCIN1/AN2/RA2): track 18.4 -> 19.5 mm
- net GND: track 109.5 -> 109.0 mm
Other:
- board text added: "Rocket Servo Rev. C1 DMFE 2024"
- board text removed: "Rocket Servo Rev. C DMFE 2024"
