File: PCB Rev C/RocketServo.kicad_sch (KiCad schematic)
At the start: 33 parts, among them IC1 PIC12F1822-I/SN, P1 Conn_01x02, P2 Conn_01x03, P3 Conn_01x02, SW1 SW_Push, SW2 SW_Push, U1 L7806, U2 L78L05_SOT89, U3 CPC1017N, U4 CPC1017N

Commit message: Rev C1
Parts:
- IC1: footprint Package_SO:SOIC-8_5.23x5.23mm_P1.27mm -> Package_SO:SOIC-8_3.9x4.9mm_P1.27mm
Other:
- note added: "Rev C1, SOIC 8 footprint changed Rev C, 6V servo power, Continuity check."
- note removed: "Rev C, 6V servo power, Continuity check."
Changed lines of the file:
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@@
 		(title "Rocket Servo")
 		(date "2024-09-23")
-		(rev "C")
+		(rev "C1")
 		(company "DMFE")
 		(comment 1 "Altimeter triggered servo")
@@
 		)
 	)
-	(text "Rev C, 6V servo power, Continuity check."
+	(text "Rev C1, SOIC 8 footprint changed\nRev C, 6V servo power, Continuity check."
 		(exclude_from_sim no)
-		(at 49.53 189.992 0)
+		(at 25.654 189.23 0)
 		(effects
 			(font
 				(size 1.524 1.524)
 			)
+			(justify left)
 		)
 	)
@@
 			)
 		)
-		(property "Footprint" "Package_SO:SOIC-8_5.23x5.23mm_P1.27mm"
+		(property "Footprint" "Package_SO:SOIC-8_3.9x4.9mm_P1.27mm"
 			(at 110.49 124.46 0)
 			(effects

Commit message: Rocket Servo 4 PCB
Other:
- note added: "R1 470Ω R2,R6,R8,R11,R12 1.0KΩ R3 10KΩ R4 220Ω R5,R7 47KΩ R9 270Ω R10 22KΩ D1 SMA 1A C1,C3,C4,C6,C7 0.1uf 0805 C2 33uf C5 220uf P2 3 pin sip pin header IC1 PIV12F1822-I/P SOIC-8 U1 L7805 DPAK U2 ua78L05 U3,U4 CPC1017N SW1,SW2 KXT341 LHS"
- note removed: "R1 470Ω R2,R6,R8,R11,R12 1.0KΩ R3 10KΩ R4 220Ω R5,R7 47KΩ R9 270Ω R10 22KΩ D1 SMA 1A C1,C3,C4,C6,C7 0.1uf 0805 C2 33uf C5 220uf P2 3 pin sip pin header IC1 PIV12F1822-I/P 8DIP U1 L7805 DPAK U2 ua78L05 U3,U4 CPC1017N 4DIP SW1,SW2 KXT341 LHS"
Changed lines of the file:
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@@
-	(wire
-		(pts
-			(xy 237.49 30.48) (xy 237.49 27.94)
-		)
-		(stroke
-			(width 0)
-			(type solid)
-		)
-	)
 	(wire
 		(pts
@@
 	(wire
 		(pts
-			(xy 232.41 30.48) (xy 237.49 30.48)
+			(xy 232.41 30.48) (xy 243.84 30.48)
 		)
 		(stroke
@@
 	(wire
 		(pts
-			(xy 237.49 27.94) (xy 252.73 27.94)
-		)
-		(stroke
-			(width 0)
-			(type solid)
-		)
-	)
-	(wire
-		(pts
 			(xy 212.09 62.23) (xy 190.5 62.23)
 		)
@@
 	(wire
 		(pts
-			(xy 252.73 109.22) (xy 196.85 109.22)
+			(xy 243.84 109.22) (xy 196.85 109.22)
 		)
 		(stroke
@@
 	(wire
 		(pts
-			(xy 252.73 27.94) (xy 252.73 109.22)
+			(xy 243.84 30.48) (xy 243.84 109.22)
 		)
 		(stroke
@@
 		)
 	)
-	(text "R1     470Ω\nR2,R6,R8,R11,R12   1.0KΩ\nR3   10KΩ\nR4   220Ω\nR5,R7   47KΩ\nR9    270Ω\nR10   22KΩ\nD1  SMA 1A\nC1,C3,C4,C6,C7  0.1uf 0805\nC2  33uf\nC5  220uf\nP2  3 pin sip pin header\nIC1 PIV12F1822-I/P 8DIP\nU1  L7805 DPAK\nU2  ua78L05\nU3,U4 CPC1017N 4DIP\nSW1,SW2 KXT341 LHS\n"
+	(text "R1     470Ω\nR2,R6,R8,R11,R12   1.0KΩ\nR3   10KΩ\nR4   220Ω\nR5,R7   47KΩ\nR9    270Ω\nR10   22KΩ\nD1  SMA 1A\nC1,C3,C4,C6,C7  0.1uf 0805\nC2  33uf\nC5  220uf\nP2  3 pin sip pin header\nIC1 PIV12F1822-I/P SOIC-8\nU1  L7805 DPAK\nU2  ua78L05\nU3,U4 CPC1017N\nSW1,SW2 KXT341 LHS\n"
 		(exclude_from_sim no)
 		(at 25.4 157.48 0)

Commit message: fixed some text
Other:
- note added: "R1 470Ω R2,R6,R8,R11,R12 1.0KΩ R3 10KΩ R4 220Ω R5,R7 47KΩ R9 270Ω R10 22KΩ D1 SMA 1A C1,C3,C4,C6,C7 0.1uf 0805 C2 33uf C5 220uf P2 3 pin sip pin header or pig-tail IC1 PIC12F1822-I/P SOIC-8 U1 L7806ABD2T D2PAK U2 ua78L05 U3,U4 CPC1017N SW1,SW2 KXT341 LHS"
- note removed: "R1 470Ω R2,R6,R8,R11,R12 1.0KΩ R3 10KΩ R4 220Ω R5,R7 47KΩ R9 270Ω R10 22KΩ D1 SMA 1A C1,C3,C4,C6,C7 0.1uf 0805 C2 33uf C5 220uf P2 3 pin sip pin header IC1 PIV12F1822-I/P SOIC-8 U1 L7805 DPAK U2 ua78L05 U3,U4 CPC1017N SW1,SW2 KXT341 LHS"
Changed lines of the file:
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@@
 		)
 	)
-	(text "R1     470Ω\nR2,R6,R8,R11,R12   1.0KΩ\nR3   10KΩ\nR4   220Ω\nR5,R7   47KΩ\nR9    270Ω\nR10   22KΩ\nD1  SMA 1A\nC1,C3,C4,C6,C7  0.1uf 0805\nC2  33uf\nC5  220uf\nP2  3 pin sip pin header\nIC1 PIV12F1822-I/P SOIC-8\nU1  L7805 DPAK\nU2  ua78L05\nU3,U4 CPC1017N\nSW1,SW2 KXT341 LHS\n"
+	(text "R1     470Ω\nR2,R6,R8,R11,R12   1.0KΩ\nR3   10KΩ\nR4   220Ω\nR5,R7   47KΩ\nR9    270Ω\nR10   22KΩ\nD1  SMA 1A\nC1,C3,C4,C6,C7  0.1uf 0805\nC2  33uf\nC5  220uf\nP2  3 pin sip pin header or pig-tail\nIC1 PIC12F1822-I/P SOIC-8\nU1  L7806ABD2T D2PAK\nU2  ua78L05\nU3,U4 CPC1017N\nSW1,SW2 KXT341 LHS\n"
 		(exclude_from_sim no)
 		(at 25.4 157.48 0)
@@
 	(label "Enable*"
 		(at 128.27 93.98 0)
-		(fields_autoplaced yes)
 		(effects
 			(font
@@
 	(label "BattV"
 		(at 152.4 116.84 0)
-		(fields_autoplaced yes)
 		(effects
 			(font

Commit message: RS2
Changed lines of the file:
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@@
 (kicad_sch
-	(version 20231120)
+	(version 20250114)
 	(generator "eeschema")
-	(generator_version "8.0")
+	(generator_version "9.0")
 	(paper "A")
 	(title_block
@@
 		(comment 1 "Altimeter triggered servo")
 	)
+	(text "+9\nGnd"
+		(exclude_from_sim no)
+		(at 63.5 34.29 0)
+		(effects
+			(font
+				(size 1.524 1.524)
+			)
+			(justify left bottom)
+		)
+	)
+	(text "R1     470Ω\nR2,R6,R8,R11,R12   1.0KΩ\nR3   10KΩ\nR4   220Ω\nR5,R7   47KΩ\nR9    270Ω\nR10   22KΩ\nD1  SMA 1A\nC1,C3,C4,C6,C7  0.1uf 0805\nC2  33uf\nC5  220uf\nP2  3 pin sip pin header or pig-tail\nIC1 PIC12F1822-I/P SOIC-8\nU1  L7806ABD2T D2PAK\nU2  ua78L05\nU3,U4 CPC1017N\nSW1,SW2 KXT341 LHS\n"
+		(exclude_from_sim no)
+		(at 25.4 157.48 0)
+		(effects
+			(font
+				(size 1.524 1.524)
+			)
+			(justify left bottom)
+		)
+	)
+	(text "Rev C1, SOIC 8 footprint changed\nRev C, 6V servo power, Continuity check."
+		(exclude_from_sim no)
+		(at 25.654 189.23 0)
+		(effects
+			(font
+				(size 1.524 1.524)
+			)
+			(justify left)
+		)
+	)
+	(text "Rev A, Added battery voltage sensing and LED connector."
+		(exclude_from_sim no)
+		(at 25.4 194.31 0)
+		(effects
+			(font
+				(size 1.524 1.524)
+			)
+			(justify left bottom)
+		)
+	)
+	(text "S\n+\n-"
+		(exclude_from_sim no)
+		(at 209.55 128.27 0)
+		(effects
+			(font
+				(size 1.524 1.524)
+			)
+			(justify right bottom)
+		)
+	)
+	(text "Trigger +\nTrigger -"
+		(exclude_from_sim no)
+		(at 64.77 64.77 0)
+		(effects
+			(font
+				(size 1.524 1.524)
+			)
+			(justify left bottom)
+		)
+	)
+	(text "Servo"
+		(exclude_from_sim no)
+		(at 208.28 118.11 0)
+		(effects
+			(font
+				(size 1.524 1.524)
+			)
+			(justify left bottom)
+		)
+	)
 	(junction
 		(at 204.47 162.56)
@@
 		)
 	)
-	(text "+9\nGnd"
-		(exclude_from_sim no)
-		(at 63.5 34.29 0)
-		(effects
-			(font
-				(size 1.524 1.524)
-			)
-			(justify left bottom)
-		)
-	)
-	(text "R1     470Ω\nR2,R6,R8,R11,R12   1.0KΩ\nR3   10KΩ\nR4   220Ω\nR5,R7   47KΩ\nR9    270Ω\nR10   22KΩ\nD1  SMA 1A\nC1,C3,C4,C6,C7  0.1uf 0805\nC2  33uf\nC5  220uf\nP2  3 pin sip pin header or pig-tail\nIC1 PIC12F1822-I/P SOIC-8\nU1  L7806ABD2T D2PAK\nU2  ua78L05\nU3,U4 CPC1017N\nSW1,SW2 KXT341 LHS\n"
-		(exclude_from_sim no)
-		(at 25.4 157.48 0)
-		(effects
-			(font
-				(size 1.524 1.524)
-			)
-			(justify left bottom)
-		)
-	)
-	(text "Rev C1, SOIC 8 footprint changed\nRev C, 6V servo power, Continuity check."
-		(exclude_from_sim no)
-		(at 25.654 189.23 0)
-		(effects
-			(font
-				(size 1.524 1.524)
-			)
-			(justify left)
-		)
-	)
-	(text "Rev A, Added battery voltage sensing and LED connector."
-		(exclude_from_sim no)
-		(at 25.4 194.31 0)
-		(effects
-			(font
-				(size 1.524 1.524)
-			)
-			(justify left bottom)
-		)
-	)
-	(text "S\n+\n-"
-		(exclude_from_sim no)
-		(at 209.55 128.27 0)
-		(effects
-			(font
-				(size 1.524 1.524)
-			)
-			(justify right bottom)
-		)
-	)
-	(text "Trigger +\nTrigger -"
-		(exclude_from_sim no)
-		(at 64.77 64.77 0)
-		(effects
-			(font
-				(size 1.524 1.524)
-			)
-			(justify left bottom)
-		)
-	)
-	(text "Servo"
-		(exclude_from_sim no)
-		(at 208.28 118.11 0)
-		(effects
-			(font
-				(size 1.524 1.524)
-			)
-			(justify left bottom)
-		)
-	)
 	(label "Enable*"
 		(at 128.27 93.98 0)
@@
 		)
 	)
+	(embedded_fonts no)
 )

Commit message: RS2
Other:
- note added: "R1 470Ω R2,R6,R8,R11,R12 1.0KΩ R3 10KΩ R4 220Ω R5,R7 47KΩ R9 270Ω R10 22KΩ D1 SMA 1A C1,C3,C4,C6,C7 0.1uf 0805 C2 33uf C5 220uf P2 3 pin sip pin header or pig-tail IC1 PIC12F1822-I/SN SOIC-8 U1 L7806ABD2T D2PAK U2 ua78L05 U3,U4 CPC1017N SW1,SW2 KXT341 LHS"
- note removed: "R1 470Ω R2,R6,R8,R11,R12 1.0KΩ R3 10KΩ R4 220Ω R5,R7 47KΩ R9 270Ω R10 22KΩ D1 SMA 1A C1,C3,C4,C6,C7 0.1uf 0805 C2 33uf C5 220uf P2 3 pin sip pin header or pig-tail IC1 PIC12F1822-I/P SOIC-8 U1 L7806ABD2T D2PAK U2 ua78L05 U3,U4 CPC1017N SW1,SW2 KXT341 LHS"
Changed lines of the file:
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@@
 		)
 	)
-	(text "R1     470Ω\nR2,R6,R8,R11,R12   1.0KΩ\nR3   10KΩ\nR4   220Ω\nR5,R7   47KΩ\nR9    270Ω\nR10   22KΩ\nD1  SMA 1A\nC1,C3,C4,C6,C7  0.1uf 0805\nC2  33uf\nC5  220uf\nP2  3 pin sip pin header or pig-tail\nIC1 PIC12F1822-I/P SOIC-8\nU1  L7806ABD2T D2PAK\nU2  ua78L05\nU3,U4 CPC1017N\nSW1,SW2 KXT341 LHS\n"
+	(text "R1     470Ω\nR2,R6,R8,R11,R12   1.0KΩ\nR3   10KΩ\nR4   220Ω\nR5,R7   47KΩ\nR9    270Ω\nR10   22KΩ\nD1  SMA 1A\nC1,C3,C4,C6,C7  0.1uf 0805\nC2  33uf\nC5  220uf\nP2  3 pin sip pin header or pig-tail\nIC1 PIC12F1822-I/SN SOIC-8\nU1  L7806ABD2T D2PAK\nU2  ua78L05\nU3,U4 CPC1017N\nSW1,SW2 KXT341 LHS\n"
 		(exclude_from_sim no)
 		(at 25.4 157.48 0)
