File: PCB RS2 Rev nc/RocketServo.kicad_sch (KiCad schematic)
At the start: 56 parts, among them J1 Conn_01x05, P1 Conn_01x02, P2 Conn_01x02, P3 Conn_01x02, P4 Conn_01x02, P5 Conn_01x02, P6 Conn_01x03, P7 Conn_01x03, P8 Conn_01x03, P9 Conn_01x03, SW1 SW_Push, SW2 SW_Push, U1 L7806, U2 L78L05_SOT89, U3 CPC1017N, U4 CPC1017N, U5 PIC16F1847-I/SO, U6 CPC1017N, U7 CPC1017N, U8 CPC1017N

Commit message: RS2
Parts:
- removed C10, C7, C9: .1uF, Capacitor_SMD:C_0805_2012Metric_Pad1.18x1.45mm_HandSolder, symbol Device:C_Small
- removed LED1, P1, P2, P3, P4, P5: Conn_01x02, Connector_PinHeader_2.54mm:PinHeader_1x02_P2.54mm_Vertical, symbol Connector_Generic:Conn_01x02
- removed P8, P9: Conn_01x03, Connector_PinHeader_2.54mm:PinHeader_1x03_P2.54mm_Vertical, symbol Connector_Generic:Conn_01x03
- removed R15: 220R, Resistor_SMD:R_0805_2012Metric_Pad1.20x1.40mm_HandSolder, symbol Device:R
- removed R18, R19: 470R, Resistor_SMD:R_0805_2012Metric_Pad1.20x1.40mm_HandSolder, symbol Device:R
- removed R25: 10K, Resistor_SMD:R_0805_2012Metric_Pad1.20x1.40mm_HandSolder, symbol Device:R
- removed U8: CPC1017N, Package_SO:SOP-4_3.8x4.1mm_P2.54mm, symbol Relay_SolidState:CPC1017N
- added C3, C4: .1uF, Capacitor_SMD:C_0805_2012Metric_Pad1.18x1.45mm_HandSolder, symbol Device:C_Small
- added D3, D4: LED, LED_SMD:LED_1206_3216Metric_Pad1.42x1.75mm_HandSolder, symbol Device:LED
- added J2: Screw_Terminal_01x08, TerminalBlock:TerminalBlock_Xinya_XY308-2.54-8P_1x08_P2.54mm_Horizontal, symbol Connector:Screw_Terminal_01x08
- added R12, R23: 1K, Resistor_SMD:R_0805_2012Metric_Pad1.20x1.40mm_HandSolder, symbol Device:R
- added R13: 2K2, Resistor_SMD:R_0805_2012Metric_Pad1.20x1.40mm_HandSolder, symbol Device:R
- added R9: 47K, Resistor_SMD:R_0805_2012Metric_Pad1.20x1.40mm_HandSolder, symbol Device:R
- added U6: LM358, Package_SO:SOIC-8_3.9x4.9mm_P1.27mm, symbol Amplifier_Operational:LM358
- R10: value 22K -> 10K
- R14: value 220R -> 100K
- R21: value 1K -> R05; footprint Resistor_SMD:R_0805_2012Metric_Pad1.20x1.40mm_HandSolder -> Resistor_SMD:R_2512_6332Metric_Pad1.40x3.35mm_HandSolder
- R6: renamed from R24; value 10K -> 1K0
- renumbered C8 to C1, C1 to C2, C2 to C5, C4 to C7, C3 to C8, C5 to C9, D2 to D1, D1 to D2, P6 to P4, P7 to P5, R9 to R15, R5 to R17, R7 to R18, R4 to R19, R13 to R20, R12 to R3, R17 to R4, R20 to R5, R3 to R7, R23 to R8, U6 to U1, U7 to U2, U1 to U7, U2 to U8
Connections:
- net Servo4 is gone; now on net Enable2: U5.3 (TOCKI/CMP2/RA4)
- net +5V: now also D3.2 (A), D4.2 (A), J2.7 (Pin_7), U6.8 (V+)
- net GND: now also R10.2, R21.2, C3.2, C4.2, J2.2 (Pin_2), R13.2, U6.4 (V-); no longer P4.3 (Pin_3), P5.3 (Pin_3), R11.1, U2.3
- net +9V: now reaches C5.1, C6.1, D2.1 (K), U7.1 (IN), U8.3 (IN)
- net +9V: now also R9.2; no longer R10.2
- net at D2.2 (A): now also J2.1 (Pin_1)
- net at U2.1: now also R6.2
- net Enable2: now reaches U2.2
- net at R15.2: now also J2.8 (Pin_8)
- net at U4.4: now also J2.4 (Pin_4)
- net at U1.2: now also U2.3
- net at R4.2: now also J2.5 (Pin_5)
- net at R1.2: now also J2.3 (Pin_3)
- net at U2.4: now also J2.6 (Pin_6); no longer R21.2
- net Servo_I: now reaches R14.1
- net Servo_I: now also U5.18 (AN1/RA1), U6.7
- net at R22.2: now also U5.10 (RB4/PGM)
- removed net BattV: R10.1, R11.2, U5.17 (AN0/RA0)
- net Enable renamed Enable1
- net Enable1: now also U5.2 (CMP1/AN3/RA3); no longer U5.18 (AN1/RA1)
- net Servo3: no longer names the net of R14.2
- net Servo3: now also R13.1, U6.6 (-); no longer U5.2 (CMP1/AN3/RA3)
- removed net Trigger3: R21.1, R6.2, U5.9 (RB3/CCP1)
- net Trigger4: no longer names the net of R22.1
- net Trigger4: now also D3.1 (K); no longer U5.10 (RB4/PGM)
- new net: R10.1, R9.1, U6.3 (+)
- new net: C3.1, R12.1, U6.5 (+)
- new net: R23.2, U5.9 (RB3/CCP1)
- new net: D4.1 (K), R23.1
- new net: R11.2, U6.1, U6.2 (-)
- new net Batt_V: C4.1, R11.1, U5.17 (AN0/RA0)
- new net GNDS: P4.3 (Pin_3), P5.3 (Pin_3), R12.2, R21.1
Other:
- note added: "10V>>1.75V"
- note added: "10mA=4.6counts"
- note added: "1A=0.05V"
- note added: "1A>>2.27V"
- note added: "LED1 + LED1 -"
- note added: "R1,R4 470Ω R2,R3,R5,R6,R11,R12,R16,R22,R23 1.0KΩ R7,R8,R10 10KΩ R9,R17,R18 47KΩ R13 2.2KΩ R14 100KΩ R15 270Ω R19,R20 220Ω R21 0.05Ω D2 SMB 2A D1,D3,D4 LED SMD1206 C1,C2,C3,C4,C6,C7,C8 0.1uf 0805 C5 33uf 25V C9 220uf 16V P1,P2,P3,LED1 2 pin sip pin header P4,P5 3 pin sip pin header U5 PID12F1847-I/SO 18SOIC U7 L7806 DPAK U8 ua78L05 U1,U2,U3,U4 CPC1017N SW1,SW2 KXT341 LHS"
- note added: "Servo 1 Active"
- note added: "Servo 2 Active"
- note added: "System LED"
- note removed: "R1,R17,R18,R19 470Ω R2,R11,R12,R16,R21,R22 1.0KΩ R3,R23,R24,R25 10KΩ R4,R13,R14,R15 220Ω R5,R7 47KΩ R9 270Ω R10 22KΩ D1 SMB 2A D2 LED SMD1206 C1,C3,C4,C6,C7,C8,C9,C10 0.1uf 0805 C2 33uf 25V C5 220uf 16V P1,P2,P3,P4,P5,LED1 2 pin sip pin header P6,P7,P8,P9 3 pin sip pin header U5 PIV12F1847-I/P 18SOIC U1 L7805 DPAK U2 ua78L05 U3,U4,U6,U7,U8 CPC1017N SW1,SW2 KXT341 LHS"
- note removed: "Trigger3 + Trigger3 -"
- note removed: "Trigger4 + Trigger4 -"
- title: Rocket Servo 4 -> Rocket Servo 2
- moved on the sheet: C1, R4, R5, R6, R8, U1, U2
