File: PCB RS2 Rev nc/RocketServo.kicad_sch (KiCad schematic)
At the start: 50 parts, among them J1 Conn_01x05, J2 Screw_Terminal_01x08, P4 Conn_01x03, P5 Conn_01x03, SW1 SW_Push, SW2 SW_Push, U1 CPC1017N, U2 CPC1017N, U3 CPC1017N, U4 CPC1017N, U5 PIC16F1847-I/SO, U6 LM358, U7 L7806, U8 L78L05_SOT89

Commit message: Two Channel Rev A
Fixed power up glitch
Other:
- note added: "0mA >> 0.003V 1C 50mA >> 0.104V 21C 500mA >> 212C"
- note added: "8.57V"
- note added: "8.79V"
- note added: "8.8V >> 1.502V 7.7V >> 1.32V 6.7V >> 1.14V"
- note added: "ADC 35.8C/V 6.5V=232C"
- note added: "R1,R4 470Ω R2,R3,R5,R6,R11,R12,R16,R22,R23 1.0KΩ R7,R8,R10 10KΩ R9,R17,R18 47KΩ R13 2.2KΩ R14 100KΩ R15 270Ω R19,R20 220Ω R21 0.05Ω 1% 2512 3W D2 SMB 2A D1,D3,D4 LED SMD1206 C1,C2,C3,C4,C6,C7,C8 0.1uf 0805 C5 33uf 25V C9 220uf 16V P1,P2,P3,LED1 2 pin sip pin header P4,P5 3 pin sip pin header U5 PIC16F1847-I/SO 18SOIC U6 LM358ADR or LM6132BIM U7 L7806 DPAK 6V 1.5A U8 ua78L05 5V 100mA U1,U2,U3,U4 C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"
- note added: "Rev. A Added notes"
- note removed: "R1,R4 470Ω R2,R3,R5,R6,R11,R12,R16,R22,R23 1.0KΩ R7,R8,R10 10KΩ R9,R17,R18 47KΩ R13 2.2KΩ R14 100KΩ R15 270Ω R19,R20 220Ω R21 0.05Ω D2 SMB 2A D1,D3,D4 LED SMD1206 C1,C2,C3,C4,C6,C7,C8 0.1uf 0805 C5 33uf 25V C9 220uf 16V P1,P2,P3,LED1 2 pin sip pin header P4,P5 3 pin sip pin header U5 PID12F1847-I/SO 18SOIC U7 L7806 DPAK U8 ua78L05 U1,U2,U3,U4 CPC1017N SW1,SW2 KXT341 LHS"
Changed lines of the file:
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@@
 		(comment 1 "Altimeter triggered servo (2 channel)")
+	)
+	(text "8.79V"
+		(exclude_from_sim no)
+		(at 145.288 28.702 0)
+		(effects
+			(font
+				(size 1.524 1.524)
+			)
+		)
 	)
 	(text "+9\nGnd"
@@
 		)
 	)
-	(text "R1,R4        470Ω\nR2,R3,R5,R6,R11,R12,R16,R22,R23 1.0KΩ\nR7,R8,R10   10KΩ\nR9,R17,R18   47KΩ\nR13           2.2KΩ\nR14           100KΩ\nR15           270Ω\nR19,R20       220Ω\nR21           0.05Ω\nD2  SMB 2A\nD1,D3,D4  LED SMD1206\nC1,C2,C3,C4,C6,C7,C8  0.1uf 0805\nC5  33uf 25V\nC9  220uf 16V\nP1,P2,P3,LED1  2 pin sip pin header\nP4,P5    3 pin sip pin header\nU5  PID12F1847-I/SO 18SOIC\nU7  L7806 DPAK\nU8  ua78L05\nU1,U2,U3,U4 CPC1017N \nSW1,SW2 KXT341 LHS\n"
+	(text "R1,R4        470Ω\nR2,R3,R5,R6,R11,R12,R16,R22,R23 1.0KΩ\nR7,R8,R10   10KΩ\nR9,R17,R18   47KΩ\nR13           2.2KΩ\nR14           100KΩ\nR15           270Ω\nR19,R20       220Ω\nR21           0.05Ω 1% 2512 3W\nD2  SMB 2A\nD1,D3,D4  LED SMD1206\nC1,C2,C3,C4,C6,C7,C8  0.1uf 0805\nC5  33uf 25V\nC9  220uf 16V\nP1,P2,P3,LED1  2 pin sip pin header\nP4,P5    3 pin sip pin header\nU5  PIC16F1847-I/SO 18SOIC\nU6  LM358ADR or LM6132BIM\nU7  L7806 DPAK 6V 1.5A\nU8  ua78L05 5V 100mA\nU1,U2,U3,U4 CPC1017N \nSW1,SW2 KXT341 LHS\nJ1 5 pin header (optional)\nJ2 8 pos screw terminal"
 		(exclude_from_sim no)
-		(at 17.526 194.31 0)
+		(at 15.494 201.168 0)
 		(effects
 			(font
@@
 		)
 	)
+	(text "Rev. A  Added notes"
+		(exclude_from_sim no)
+		(at 238.76 170.434 0)
+		(effects
+			(font
+				(size 1.524 1.524)
+			)
+		)
+	)
 	(text "10V>>1.75V"
 		(exclude_from_sim no)
 		(at 155.194 58.166 0)
+		(effects
+			(font
+				(size 1.524 1.524)
+			)
+		)
+	)
+	(text "0mA >> 0.003V 1C\n50mA >> 0.104V 21C\n500mA >> 212C"
+		(exclude_from_sim no)
+		(at 179.324 85.852 0)
 		(effects
 			(font
@@
 		)
 	)
+	(text "8.57V"
+		(exclude_from_sim no)
+		(at 178.054 28.956 0)
+		(effects
+			(font
+				(size 1.524 1.524)
+			)
+		)
+	)
 	(text "LED1 +\nLED1 -"
 		(exclude_from_sim no)
@@
 		(effects
 			(font
+				(size 1.524 1.524)
+			)
+		)
+	)
+	(text "8.8V >> 1.502V\n7.7V >> 1.32V\n6.7V >> 1.14V"
+		(exclude_from_sim no)
+		(at 169.926 63.754 0)
+		(effects
+			(font
+				(size 1.524 1.524)
+			)
+		)
+	)
+	(text "ADC 35.8C/V  6.5V=232C"
+		(exclude_from_sim no)
+		(at 176.784 106.68 0)
+		(effects
+			(font
